File: Displej/BT_displej_rizeni_v3.brd (EAGLE design)
At the start: 54 x 34.3 mm, 48 parts, among them IC1 MCP1703DB, Q1 8MHz, Q2 BSS123, Q3 BSS123, X7 ARK500/2EX, X8 MINI-USB-32005-201

Commit message: new file:   Ctecka/ctecka_brana.brd 	new file:   Ctecka/ctecka_brana.sch 	new file:   Ctecka/ctecka_mala.brd 	new file:   Ctecka/ctecka_mala.sch 	new file:   Ctecka/ctecka_stolni.brd 	new file:   Ctecka/ctecka_stolni.sch 	modified:   Displej/BT_displej_rizeni_v2.brd 	modified:   Displej/BT_displej_rizeni_v2.sch 	new file:   Displej/BT_displej_rizeni_v3.brd 	new file:   Displej/BT_displej_rizeni_v3.sch
Parts:
- removed C12, C13: 15p, rcl:C0603
- removed C14: 10n, rcl:C0603
- removed C15, C16, C21: 100n, rcl:C0603
- removed C9: 1u, rcl:C0603
- removed D7: 1N4148SMD, diode:MINIMELF
- removed Q1: 8MHz, crystal:CTS406
- removed R14: 4k7, rcl:R0603
- removed R19, R42: 10k, rcl:R0603
- removed R4, R9: 22R, rcl:R0603
- removed R41: 5k1, rcl:R0603
- removed S1, S2: TSHA-2P(docasne), switch-tact:DTSM-3
- removed U$3: ATMEGA8U2, atmel:VQFP32
- removed X8: MINI-USB-32005-201, con-cypressindustries:32005-201
- added C10, C19, C20: (no value), rcl:C0603
- added IC3: MEGA8-AI, atmel:TQFP32-08
- added Q4: (no value), crystal:CTS406
- added R3: (no value), rcl:R0603
- added TP1, TP2, TP3, TP4, TP5, TP6: TPB1,27, testpad:B1,27
Connections:
- removed net 323: R19.1, S1.1, U$3.13
- removed net N$14: C13.2, Q1.3, U$3.2
- removed net N$16: R9.1, X8.3
- removed net N$17: R4.2, U$3.30
- removed net N$18: R9.2, U$3.29
- removed net N$19: R41.1, R42.2, U$3.26
- removed net N$63: C9.1, U$3.27
- removed net N$64: C21.1, R41.2, X8.1
- removed net N$7: C12.2, Q1.1, U$3.1
- removed net N$8: R4.1, X8.2
- removed net RESET: C14.1, D7.A, R14.1, S2.2, U$3.24
- removed net USB_4: X8.4
- new net +5V: IC3.18, IC3.20, IC3.4, IC3.6, R3.1, TP2.TP
- new net N$39: C10.1, IC3.8, Q4.3
- new net N$40: C19.1, IC3.7, Q4.1
- new net N$44: C20.2, IC3.29, R3.2, TP6.TP
- net +3V3: no longer C15.2, C16.2, D7.C, R14.2, R19.2, U$3.31, U$3.32, U$3.4
- net GND: now also C10.2, C19.2, C20.1, IC3.21, IC3.3, IC3.5, TP1.TP; no longer C12.1, C13.1, C14.2, C15.1, C16.1, C21.2, C9.2, R42.1, S1.2, S2.1, U$3.28, U$3.3, X8.5
- net N$1: no longer U$3.8
- net N$10: no longer U$3.6
- net N$11: no longer U$3.7
- net N$24: now also IC3.14; no longer U$3.14
- net N$27: now also IC3.17, TP3.TP; no longer U$3.15
- net N$28: now also IC3.15, TP5.TP; no longer U$3.16
- net N$29: now also IC3.16, TP4.TP; no longer U$3.17
- net N$5: no longer U$3.9
Routing:
- net +3V3: track 65.3 -> 33.8 mm, vias 3 -> 1
- net N$19: track 13.0 -> 0.00 mm, vias 1 -> 0
- net RESET: track 12.5 -> 0.00 mm, vias 1 -> 0
- net N$7: track 8.72 -> 0.00 mm
- net 323: track 8.15 -> 0.00 mm, vias 1 -> 0
- net N$64: track 8.13 -> 0.00 mm
- net N$5: track 29.6 -> 22.6 mm
- net N$14: track 5.88 -> 0.00 mm
- net N$1: track 28.6 -> 22.9 mm
- net N$18: track 3.21 -> 0.00 mm, vias 1 -> 0
- net N$16: track 3.08 -> 0.00 mm
- net N$8: track 2.88 -> 0.00 mm
- net N$17: track 2.83 -> 0.00 mm, vias 1 -> 0
- net GND: track 2.74 -> 0.00 mm, vias 125 -> 124
- net N$28: track 24.4 -> 22.5 mm
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