File: Displej/BT_displej_rizeni_v3.sch (EAGLE design)
At the start: 48 parts, among them IC1 MCP1703DB, Q1 8MHz, Q2 BSS123, Q3 BSS123, X7 ARK500/2EX, X8 MINI-USB-32005-201

Commit message: new file:   Ctecka/ctecka_brana.brd 	new file:   Ctecka/ctecka_brana.sch 	new file:   Ctecka/ctecka_mala.brd 	new file:   Ctecka/ctecka_mala.sch 	new file:   Ctecka/ctecka_stolni.brd 	new file:   Ctecka/ctecka_stolni.sch 	modified:   Displej/BT_displej_rizeni_v2.brd 	modified:   Displej/BT_displej_rizeni_v2.sch 	new file:   Displej/BT_displej_rizeni_v3.brd 	new file:   Displej/BT_displej_rizeni_v3.sch
Parts:
- removed C12, C13: 15p, rcl:C-EUC0603
- removed C14: 10n, rcl:C-EUC0603
- removed C15, C16, C21: 100n, rcl:C-EUC0603
- removed C9: 1u, rcl:C-EUC0603
- removed D7: 1N4148SMD, diode:DIODE-MINIMELF
- removed Q1: 8MHz, crystal:CRYSTALCTS406
- removed R14: 4k7, rcl:R-EU_R0603
- removed R19, R42: 10k, rcl:R-EU_R0603
- removed R4, R9: 22R, rcl:R-EU_R0603
- removed R41: 5k1, rcl:R-EU_R0603
- removed S1, S2: TSHA-2P(docasne), switch-tact:DTSM-3
- removed U$3: ATMEGA8U2, atmel:ATMEGA8U2
- removed X8: MINI-USB-32005-201, con-cypressindustries:MINI-USB-32005-201
- added C10, C19, C20: (no value), rcl:C-EUC0603
- added IC3: MEGA8-AI, atmel:MEGA8-AI
- added Q4: (no value), crystal:CRYSTALCTS406
- added R3: (no value), rcl:R-EU_R0603
- added TP1, TP2, TP3, TP4, TP5, TP6: TPB1,27, testpad:TPB1,27
Connections:
- removed net 323: R19.1, S1.1, U$3.(!CTS!/!HWB!/AIN6/T0/INT7)PD7
- removed net N$14: C13.2, Q1.2, U$3.XTAL2(PC0)
- removed net N$16: R9.1, X8.3
- removed net N$17: R4.2, U$3.D-
- removed net N$18: R9.2, U$3.D+
- removed net N$19: R41.1, R42.2, U$3.(PCINT10)PC4
- removed net N$63: C9.1, U$3.UCAP
- removed net N$64: C21.1, R41.2, X8.1
- removed net N$7: C12.2, Q1.1, U$3.XTAL1
- removed net N$8: R4.1, X8.2
- removed net RESET: C14.1, D7.A, R14.1, S2.2, U$3.!RESET!(PC1/DW)
- removed net USB_4: X8.4
- new net +5V: IC3.AREF, IC3.AVCC, IC3.VCC@1, IC3.VCC@2, R3.1, TP2.TP
- new net N$39: C10.1, IC3.PB7(XTAL2/TOSC2), Q4.2
- new net N$40: C19.1, IC3.PB6(XTAL1/TOSC1), Q4.1
- new net N$44: C20.2, IC3.PC6(/RESET), R3.2, TP6.TP
- net +3V3: no longer C15.2, C16.2, D7.C, R14.2, R19.2, U$3.AVCC, U$3.UVCC, U$3.VCC
- net GND: now also C10.2, C19.2, C20.1, IC3.GND, IC3.GND@1, IC3.GND@2, TP1.TP; no longer C12.1, C13.1, C14.2, C15.1, C16.1, C21.2, C9.2, R42.1, S1.2, S2.1, U$3.GND, U$3.UGND, X8.5
- net N$1: no longer U$3.(ANI1/RXD1/INT2)PD2
- net N$10: no longer U$3.(OC0B/INT0)PD0
- net N$11: no longer U$3.(AIN0/SDA/INT1)PD1
- net N$24: now also IC3.PB2(SS/OC1B); no longer U$3.(!SS!/PCINT0)PB0
- net N$27: now also IC3.PB5(SCK), TP3.TP; no longer U$3.(PCINT1/SCLK)PB1
- net N$28: now also IC3.PB3(MOSI/OC2), TP5.TP; no longer U$3.(PDI/PCINT2/MOSI)PB2
- net N$29: now also IC3.PB4(MISO), TP4.TP; no longer U$3.(PDO/PCINT3/MISO)PB3
- net N$5: no longer U$3.(TXD1/INT3)PD3
